File: pcb/nodo edge IIot.kicad_sch (KiCad schematic)
At the start: 11 parts, among them J1 ESP32_DEVKIT_38P, J2 PZEM_004T, J3 DC_IN

Commit message: Update PCB design
Parts:
- removed J1: ESP32_DEVKIT_38P, Esp 38 pin:ESP32-38pin, symbol Connector_Generic:Conn_02x19_Odd_Even
- added ESP32_38P1: ~, Esp 38 pin:ESP32-38pin, symbol ESP32-38pin:Esp32
Connections:
- net GND: now also ESP32_38P1.14 (GND)
- net GPIO21: now also ESP32_38P1.33 (GPIO21)
- net GPIO22: now also ESP32_38P1.36 (GPIO22)
- net GPIO23: now also ESP32_38P1.37 (GPIO23)
- net RX_PZEM: now also ESP32_38P1.27 (GPIO16)
- net TX_PZEM: now also ESP32_38P1.28 (GPIO17)
- net VIN: now also ESP32_38P1.19 (5V)
- no-connect marks 32 -> 34
